Commit message: Add files via upload

File: sawyer_robot/sawyer_description/urdf/human.urdf (robot description, URDF)
Before this commit: robot dumpUrdf, 17 links, 16 joints
Joints:
- joint left_shoulder: limit lower=-3.14 upper=3.14 effort=1000.0 velocity=0.5 -> (none); type revolute -> continuous
- joint right_shoulder: limit lower=-3.14 upper=3.14 effort=1000.0 velocity=0.5 -> (none); type revolute -> continuous
